File: BajaBlaster/BajaBlaster.kicad_sch (KiCad schematic)
At the start: 14 parts, among them J1 Conn_01x02_Pin, U1 ESP32-WROOM-32, U2 TPS562200, U3 AP2112K-3.3

Commit message: added seperate subsections
Parts:
- removed C1: 100nF, symbol Device:C
- removed C2: 10uF, symbol Device:C
- removed C3: 22uF, symbol Device:C
- removed C4, C5: 1uF, symbol Device:C
- removed F1: Fuse, symbol Device:Fuse
- removed J1: Conn_01x02_Pin, symbol Connector:Conn_01x02_Pin
- removed L1: 22uH, symbol Device:L
- removed R1, R2: 100kOHM, symbol Device:R
- removed R3: 18.7kOHM, symbol Device:R
- removed U1: ESP32-WROOM-32, RF_Module:ESP32-WROOM-32, symbol RF_Module:ESP32-WROOM-32
- removed U2: TPS562200, Package_TO_SOT_SMD:SOT-23-6, symbol Regulator_Switching:TPS562200
- removed U3: AP2112K-3.3, Package_TO_SOT_SMD:SOT-23-5, symbol Regulator_Linear:AP2112K-3.3
Other:
- added sheet COMMS (comms.kicad_sch)
- added sheet MCU (mcu.kicad_sch)
- added sheet POWER (power.kicad_sch)
- added sheet SENSORS (sensors.kicad_sch)
