File: BajaBlaster/comms.kicad_sch (KiCad schematic)
At the start: 1 part

Commit message: moved
Parts:
- renumbered J to J2
Other:
- moved on the sheet: J2
Changed lines of the file:
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@@
 	(text "PROGRAMMING HEADER"
 		(exclude_from_sim no)
-		(at 12.3272 1.0216 0)
-		(effects
-			(font
-				(size 1.27 1.27)
-			)
-		)
-	)
-	(wire
-		(pts
-			(xy 28.8372 8.1336) (xy 28.8372 10.6736)
-		)
-		(stroke
-			(width 0)
-			(type default)
-		)
-	)
-	(wire
-		(pts
-			(xy 12.3272 13.2136) (xy 28.8372 13.2136)
-		)
-		(stroke
-			(width 0)
-			(type default)
-		)
-	)
-	(wire
-		(pts
-			(xy 12.3272 18.2936) (xy 14.8672 18.2936)
-		)
-		(stroke
-			(width 0)
-			(type default)
-		)
-	)
-	(wire
-		(pts
-			(xy 28.8372 10.6736) (xy 12.3272 10.6736)
-		)
-		(stroke
-			(width 0)
-			(type default)
-		)
-	)
-	(wire
-		(pts
-			(xy 12.3272 20.8336) (xy 14.8672 20.8336)
-		)
-		(stroke
-			(width 0)
-			(type default)
-		)
-	)
-	(wire
-		(pts
-			(xy 28.8372 13.2136) (xy 28.8372 15.7536)
-		)
-		(stroke
-			(width 0)
-			(type default)
-		)
-	)
-	(wire
-		(pts
-			(xy 12.3272 15.7536) (xy 14.8672 15.7536)
-		)
-		(stroke
-			(width 0)
-			(type default)
-		)
-	)
-	(wire
-		(pts
-			(xy 12.3272 23.3736) (xy 14.8672 23.3736)
+		(at 41.91 32.258 0)
+		(effects
+			(font
+				(size 1.27 1.27)
+			)
+		)
+	)
+	(wire
+		(pts
+			(xy 58.42 39.37) (xy 58.42 41.91)
+		)
+		(stroke
+			(width 0)
+			(type default)
+		)
+	)
+	(wire
+		(pts
+			(xy 41.91 44.45) (xy 58.42 44.45)
+		)
+		(stroke
+			(width 0)
+			(type default)
+		)
+	)
+	(wire
+		(pts
+			(xy 41.91 49.53) (xy 44.45 49.53)
+		)
+		(stroke
+			(width 0)
+			(type default)
+		)
+	)
+	(wire
+		(pts
+			(xy 58.42 41.91) (xy 41.91 41.91)
+		)
+		(stroke
+			(width 0)
+			(type default)
+		)
+	)
+	(wire
+		(pts
+			(xy 41.91 52.07) (xy 44.45 52.07)
+		)
+		(stroke
+			(width 0)
+			(type default)
+		)
+	)
+	(wire
+		(pts
+			(xy 58.42 44.45) (xy 58.42 46.99)
+		)
+		(stroke
+			(width 0)
+			(type default)
+		)
+	)
+	(wire
+		(pts
+			(xy 41.91 46.99) (xy 44.45 46.99)
+		)
+		(stroke
+			(width 0)
+			(type default)
+		)
+	)
+	(wire
+		(pts
+			(xy 41.91 54.61) (xy 44.45 54.61)
 		)
 		(stroke
@@
 	)
 	(label "IO1"
-		(at 14.8672 15.7536 0)
+		(at 44.45 46.99 0)
 		(effects
 			(font
@@
 	)
 	(label "IO3"
-		(at 14.8672 18.2936 0)
+		(at 44.45 49.53 0)
 		(effects
 			(font
@@
 	)
 	(label "IO0"
-		(at 14.8672 23.3736 0)
+		(at 44.45 54.61 0)
 		(effects
 			(font
@@
 	)
 	(label "ESP32 EN"
-		(at 14.8672 20.8336 0)
+		(at 44.45 52.07 0)
 		(effects
 			(font
@@
 	(symbol
 		(lib_id "power:GND")
-		(at 28.8372 15.7536 0)
+		(at 58.42 46.99 0)
 		(unit 1)
 		(body_style 1)
@@
 		(dnp no)
 		(fields_autoplaced yes)
-		(property "Reference" "#PWR"
-			(at 28.8372 22.1036 0)
+		(property "Reference" "#PWR018"
+			(at 58.42 53.34 0)
 			(hide yes)
 			(show_name no)
@@
 		)
 		(property "Value" "GND"
-			(at 28.8372 20.8336 0)
+			(at 58.42 52.07 0)
 			(show_name no)
 			(do_not_autoplace no)
@@
 		)
 		(property "Footprint" ""
-			(at 28.8372 15.7536 0)
+			(at 58.42 46.99 0)
 			(hide yes)
 			(show_name no)
@@
 		)
 		(property "Datasheet" ""
-			(at 28.8372 15.7536 0)
+			(at 58.42 46.99 0)
 			(hide yes)
 			(show_name no)
@@
 		)
 		(property "Description" "Power symbol creates a global label with name \"GND\" , ground"
-			(at 28.8372 15.7536 0)
+			(at 58.42 46.99 0)
 			(hide yes)
 			(show_name no)
@@
 		(instances
 			(project "BajaBlaster"
-				(path "/08a0edf5-ad57-4ef4-97bf-c48cb466bb64"
+				(path "/08a0edf5-ad57-4ef4-97bf-c48cb466bb64/a8b20a94-9e87-4c03-83c5-8129ea634c32"
 					(reference "#PWR018")
 					(unit 1)
@@
 	(symbol
 		(lib_id "Connector:Conn_01x06_Pin")
-		(at 7.2472 15.7536 0)
+		(at 36.83 46.99 0)
 		(unit 1)
 		(body_style 1)
@@
 		(dnp no)
 		(fields_autoplaced yes)
-		(property "Reference" "J"
-			(at 7.8822 5.5936 0)
+		(property "Reference" "J2"
+			(at 37.465 36.83 0)
 			(show_name no)
 			(do_not_autoplace no)
@@
 		)
 		(property "Value" "Conn_01x06_Pin"
-			(at 7.8822 8.1336 0)
+			(at 37.465 39.37 0)
 			(show_name no)
 			(do_not_autoplace no)
@@
 		)
 		(property "Footprint" ""
-			(at 7.2472 15.7536 0)
+			(at 36.83 46.99 0)
 			(hide yes)
 			(show_name no)
@@
 		)
 		(property "Datasheet" ""
-			(at 7.2472 15.7536 0)
+			(at 36.83 46.99 0)
 			(hide yes)
 			(show_name no)
@@
 		)
 		(property "Description" "Generic connector, single row, 01x06, script generated"
-			(at 7.2472 15.7536 0)
+			(at 36.83 46.99 0)
 			(hide yes)
 			(show_name no)
@@
 		(instances
 			(project "BajaBlaster"
-				(path "/08a0edf5-ad57-4ef4-97bf-c48cb466bb64"
+				(path "/08a0edf5-ad57-4ef4-97bf-c48cb466bb64/a8b20a94-9e87-4c03-83c5-8129ea634c32"
 					(reference "J2")
 					(unit 1)
@@
 	(symbol
 		(lib_id "power:+3V3")
-		(at 28.8372 8.1336 0)
+		(at 58.42 39.37 0)
 		(unit 1)
 		(body_style 1)
@@
 		(dnp no)
 		(fields_autoplaced yes)
-		(property "Reference" "#PWR"
-			(at 28.8372 11.9436 0)
+		(property "Reference" "#PWR017"
+			(at 58.42 43.18 0)
 			(hide yes)
 			(show_name no)
@@
 		)
 		(property "Value" "+3V3"
-			(at 28.8372 3.0536 0)
+			(at 58.42 34.29 0)
 			(show_name no)
 			(do_not_autoplace no)
@@
 		)
 		(property "Footprint" ""
-			(at 28.8372 8.1336 0)
+			(at 58.42 39.37 0)
 			(hide yes)
 			(show_name no)
@@
 		)
 		(property "Datasheet" ""
-			(at 28.8372 8.1336 0)
+			(at 58.42 39.37 0)
 			(hide yes)
 			(show_name no)
@@
 		)
 		(property "Description" "Power symbol creates a global label with name \"+3V3\""
-			(at 28.8372 8.1336 0)
+			(at 58.42 39.37 0)
 			(hide yes)
 			(show_name no)
@@
 		(instances
 			(project "BajaBlaster"
-				(path "/08a0edf5-ad57-4ef4-97bf-c48cb466bb64"
+				(path "/08a0edf5-ad57-4ef4-97bf-c48cb466bb64/a8b20a94-9e87-4c03-83c5-8129ea634c32"
 					(reference "#PWR017")
 					(unit 1)
