File: BajaBlaster/comms.kicad_sch (KiCad schematic)
At the start: 7 parts, among them J501 Conn_01x06_Pin, J502 INTERBOARD, J503 Conn_01x04_Pin, U501 TCAN330

Commit message: sendoff
Parts:
- removed J502: INTERBOARD, Connector_Molex:Molex_Micro-Fit_3.0_43045-0610_2x03-1MP_P3.00mm_Horizontal, symbol Connector_Generic:Conn_02x03_Odd_Even
- added C502: 100nf, Capacitor_SMD:C_0805_2012Metric, symbol Device:C
- added C503, C504, C505, C506, C507, C508, C509, C510: 47pF 50V, Capacitor_SMD:C_0805_2012Metric, symbol Device:C
- added D501, D502: NUP2105L, Package_TO_SOT_SMD:SOT-23, symbol Power_Protection:NUP2105L
- added FL501, FL502: 1812CAN-513NRC, Inductor_SMD:L_CommonModeChoke_Coilcraft_1812CAN, symbol Device:Filter_EMI_LL_1423
- added J502, J504: Conn_01x04_Pin, Connector_JST:JST_JWPF_B04B-JWPF-SK-R_1x04_P2.00mm_Vertical, symbol Connector:Conn_01x04_Pin
- added JP502: SolderJumper_2_Open, Jumper:SolderJumper-2_P1.3mm_Open_Pad1.0x1.5mm, symbol Jumper:SolderJumper_2_Open
- added JP503: JP_EXT_PWR, Jumper:SolderJumper-2_P1.3mm_Open_Pad1.0x1.5mm, symbol Jumper:SolderJumper_2_Open
- added R_CAN_TERM502: 120 OHM, Resistor_SMD:R_0805_2012Metric, symbol Device:R
- added U502: TCAN330, Package_SO:SOIC-8_3.9x4.9mm_P1.27mm, symbol Interface_CAN_LIN:TCAN330
- J503: footprint Connector_Molex:Molex_Micro-Fit_3.0_43650-0412_1x04-1MP_P3.00mm_Horizontal -> Connector_JST:JST_JWPF_B04B-JWPF-SK-R_1x04_P2.00mm_Vertical
Connections:
- net +3V3: now also C502.2, U502.3 (VCC)
- net GND: now also C502.1, C503.2, C504.2, C505.2, C506.2, C507.2, C508.2, C509.2, C510.2, D501.3 (A), D502.3 (A), J502.2 (Pin_2), J504.2 (Pin_2), U502.2 (GND), U502.5 (SHDN), U502.8 (S)
- net +12V: no longer names the net of J503.1 (Pin_1)
- net +12V: now also JP503.1 (A)
- removed net CANH: J503.3 (Pin_3), R_CAN_TERM501.1, U501.7 (CANH)
- removed net CANL: J503.4 (Pin_4), JP501.2 (B), U501.6 (CANL)
- net CAN_RX renamed EXT_CAN_RX
- net CAN_TX renamed EXT_CAN_TX
- net ESP32_EN renamed NRST
- net IO0 renamed SWO
- net U0RXD renamed SWCLK
- net U0TXD renamed SWDIO
- new net: JP502.1 (A), R_CAN_TERM502.2
- new net EXT_5V_IN: J502.1 (Pin_1), J504.1 (Pin_1), JP503.2 (B)
- new net EXT_CAN_H: C506.1, D501.2 (K), FL501.3, J503.3 (Pin_3), R_CAN_TERM502.1
- new net EXT_CAN_H_IC: C503.1, FL501.2, U501.7 (CANH)
- new net EXT_CAN_L: C505.1, D501.1 (K), FL501.4, J503.4 (Pin_4), JP502.2 (B)
- new net EXT_CAN_L_IC: C504.1, FL501.1, U501.6 (CANL)
- new net INTER_CAN_H: C510.1, D502.2 (K), FL502.3, J502.3 (Pin_3), J504.3 (Pin_3), R_CAN_TERM501.1
- new net INTER_CAN_H_IC: C508.1, FL502.2, U502.7 (CANH)
- new net INTER_CAN_L: C509.1, D502.1 (K), FL502.4, J502.4 (Pin_4), J504.4 (Pin_4), JP501.2 (B)
- new net INTER_CAN_L_IC: C507.1, FL502.1, U502.6 (CANL)
- new net INTER_CAN_RX: U502.4 (RXD)
- new net INTER_CAN_TX: U502.1 (TXD)
Other:
- note added: "CAN EMI FILTERS"
- note added: "EXT CAN CONNECTOR"
- note added: "EXT CAN TRANCIEVER"
- note added: "INTER CAN CONNECTORS"
- note added: "INTER CAN TRANCIEVER"
- note removed: "CAN CONNECTOR"
- note removed: "CAN TRANSCEIVER"
- note removed: "INTERBOARD CONNECTOR"
- moved on the sheet: C501, J503, JP501, R_CAN_TERM501, U501
