File: BajaBlaster/BajaBlaster.kicad_pcb (KiCad board)
At the start: 4 copper layers, 14 parts, among them J301 Conn_01x06_Socket, J502 INTERBOARD, SW301 SW_Push, U201 AP2112K-3.3, U202 TPS562200, U301 ESP32-WROOM-32, U302 MPU-6050

Commit message: added all the footprints - no errors - dont know if they are correct yet though
Parts:
- removed C302: 10uF, Package_SO:SOIC-8_3.9x4.9mm_P1.27mm
- removed C304: 0.1uF, Package_SO:SOIC-8_3.9x4.9mm_P1.27mm
- removed C305: 0.1uf, Package_SO:SOIC-8_3.9x4.9mm_P1.27mm
- removed C306: 2.2nf, Package_SO:SOIC-8_3.9x4.9mm_P1.27mm
- removed J301: Conn_01x06_Socket, Connector:Tag-Connect_TC2030-IDC-FP_2x03_P1.27mm_Vertical
- removed J502: INTERBOARD, Package_DFN_QFN:QFN-20-1EP_5x5mm_P0.65mm_EP3.35x3.35mm
- removed R303: 10kOhm, Package_DIP:DIP-8_W7.62mm
- removed R304, R305: 4.7kOHM, Package_DIP:DIP-8_W7.62mm
- removed SW301: SW_Push, Package_DIP:DIP-24_W7.62mm
- removed U201: AP2112K-3.3, Package_TO_SOT_SMD:SOT-23-5
- removed U202: TPS562200, Package_TO_SOT_SMD:SOT-23-6
- removed U301: ESP32-WROOM-32, RF_Module:ESP32-WROOM-32
- removed U302: MPU-6050, Sensor_Motion:InvenSense_QFN-24_4x4mm_P0.5mm

Commit message: made the ground plane
Parts:
- added C201: 1uF, Capacitor_SMD:C_0805_2012Metric, F.Cu at (87.9, -27.2)
- added C202: 100uF, Capacitor_SMD:C_0805_2012Metric, F.Cu at (87.9, -24.2)
- added C203: 1uF, Capacitor_SMD:C_0805_2012Metric, F.Cu at (87.9, -21.2)
- added C204: 10uF, Capacitor_SMD:C_0805_2012Metric, F.Cu at (87.9, -18.2)
- added C205: 22uF, Capacitor_SMD:C_0805_2012Metric, F.Cu at (87.9, -15.2)
- added C206: 100nF, Capacitor_SMD:C_0805_2012Metric, F.Cu at (87.9, -12.1)
- added C301: 1uF, Capacitor_SMD:C_0805_2012Metric, F.Cu at (69.8, -57.5)
- added C302: 10uF, Capacitor_SMD:C_0805_2012Metric, F.Cu at (69.8, -54.5)
- added C303: 100nF, Capacitor_SMD:C_0805_2012Metric, F.Cu at (69.8, -51.5)
- added C304: 0.1uF, Capacitor_SMD:C_0805_2012Metric, F.Cu at (69.8, -48.5)
- added C305: 0.1uf, Capacitor_SMD:C_0805_2012Metric, F.Cu at (69.8, -45.5)
- added C306: 2.2nf, Capacitor_SMD:C_0805_2012Metric, F.Cu at (69.8, -42.4)
- added C501: 100nf, Capacitor_SMD:C_0805_2012Metric, F.Cu at (96.0, -47.4)
- added D201: SMBJ24A, Diode_SMD:D_SMB, F.Cu at (94.4, -9.12)
- added F201: Fuse, Fuse:Fuse_1206_3216Metric, F.Cu at (81.2, -13.5)
- added J201: Conn_01x02_Pin, Connector_Molex:Molex_Micro-Fit_3.0_43650-0210_1x02-1MP_P3.00mm_Horizontal, F.Cu at (79.9, -22.7)
- added J301: Conn_01x06_Socket, Connector:Tag-Connect_TC2030-IDC-FP_2x03_P1.27mm_Vertical, F.Cu at (32.8, -11.9)
- added J501: Conn_01x06_Pin, Connector_PinHeader_2.54mm:PinHeader_1x06_P2.54mm_Vertical, F.Cu at (76.3, -56.7)
- added J502: INTERBOARD, Connector_Molex:Molex_Micro-Fit_3.0_43045-0600_2x03_P3.00mm_Horizontal, F.Cu at (83.2, -49.1)
- added J503: Conn_01x04_Pin, Connector_Molex:Molex_Micro-Fit_3.0_43650-0410_1x04-1MP_P3.00mm_Horizontal, F.Cu at (87.4, -38.3)
- added JP501: SolderJumper_2_Open, Jumper:SolderJumper-2_P1.3mm_Open_Pad1.0x1.5mm, F.Cu at (96.0, -50.6)
- added L201: 22uH, Inductor_SMD:L_Bourns_SRN6045TA, F.Cu at (94.0, -25.5)
- added R201: 100kOHM, Resistor_SMD:R_0805_2012Metric, F.Cu at (76.2, -13.6)
- added R202: 100kOHM, Resistor_SMD:R_0805_2012Metric, F.Cu at (76.2, -10.7)
- added R203: 18.7kOHM, Resistor_SMD:R_0805_2012Metric, F.Cu at (76.2, -7.75)
- added R301: 10kOHM, Resistor_SMD:R_0805_2012Metric, F.Cu at (69.8, -39.5)
- added R302: 50 OHM, Resistor_SMD:R_0805_2012Metric, F.Cu at (69.8, -36.5)
- added R303: 10kOhm, Resistor_SMD:R_0805_2012Metric, F.Cu at (69.8, -33.6)
- added R304: 4.7kOHM, Resistor_SMD:R_0805_2012Metric, F.Cu at (69.8, -30.6)
- added R305: 4.7kOHM, Resistor_SMD:R_0805_2012Metric, F.Cu at (69.8, -27.7)
- added R_CAN_TERM501: 120 OHM, Resistor_SMD:R_0805_2012Metric, F.Cu at (98.5, -42.8)
- added SW301: SW_Push, Button_Switch_SMD:SW_SPST_TL3342, F.Cu at (23.3, -13.2)
- added SW302: SW_Push, Button_Switch_SMD:SW_SPST_TL3342, F.Cu at (23.3, -6.12)
- added U201: AP2112K-3.3, Package_TO_SOT_SMD:SOT-23-5, F.Cu at (92.7, -18.8)
- added U202: TPS562200, Package_TO_SOT_SMD:SOT-23-6, F.Cu at (92.7, -14.1)
- added U301: ESP32-WROOM-32, RF_Module:ESP32-WROOM-32, F.Cu at (73.4, 41.4)
- added U302: MPU-6050, Sensor_Motion:InvenSense_QFN-24_4x4mm_P0.5mm, F.Cu at (40.3, -13.5)
- added U501: TCAN330, Package_SO:SOIC-8_3.9x4.9mm_P1.27mm, F.Cu at (98.0, -55.6)
Other:
- board outline added: 60 x 50 mm

Commit message: small tweaks
Parts:
- added REF**: MountingHole_3.2mm_M3_ISO14580_Pad, MountingHole:MountingHole_3.2mm_M3_ISO14580_Pad, F.Cu at (116.0, 35.5)
- added REF**: MountingHole_3.2mm_M3_ISO14580_Pad, MountingHole:MountingHole_3.2mm_M3_ISO14580_Pad, F.Cu at (48.5, 96.0)
- added REF**: MountingHole_3.2mm_M3_ISO14580_Pad, MountingHole:MountingHole_3.2mm_M3_ISO14580_Pad, F.Cu at (116.0, 96.0)
- added REF**: MountingHole_3.2mm_M3_ISO14580_Pad, MountingHole:MountingHole_3.2mm_M3_ISO14580_Pad, F.Cu at (48.5, 35.5)
- J301: footprint Connector:Tag-Connect_TC2030-IDC-FP_2x03_P1.27mm_Vertical -> Connector_PinHeader_2.54mm:PinHeader_1x06_P2.54mm_Vertical_SMD_Pin1Left
- moved U501 145.3 mm to (110.8, 89.1)
- moved J501 122.2 mm to (87.4, 65.0), turned to 90 degrees
- moved U302 116.0 mm to (97.8, 87.2)
- moved L201 114.0 mm to (51.0, 80.1), turned to 90 degrees
- moved J502 113.4 mm to (108.5, 61.5), turned to -90 degrees
- moved J301 104.0 mm to (93.7, 72.3), turned to 90 degrees
- moved SW302 99.6 mm to (99.6, 57.9)
- moved C205 97.6 mm to (61.2, 78.8)
- moved SW301 95.4 mm to (86.9, 57.9)
- moved C206 93.3 mm to (51.0, 73.5), turned to 90 degrees
- moved U201 92.4 mm to (72.0, 71.2)
- moved J503 90.1 mm to (112.4, 48.2), turned to -90 degrees
- moved U202 88.2 mm to (57.7, 66.9), turned to -90 degrees
- moved R202 84.3 mm to (57.0, 71.4), turned to 90 degrees
- moved C202 80.9 mm to (69.3, 54.5)
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Routing:
- net GND: track 0.00 -> 16.0 mm, vias 0 -> 8
- net /POWER/VREG_EN: track 0.00 -> 10.3 mm
- net +12V: track 0.00 -> 9.91 mm, vias 0 -> 4
- net Net-(U202-VFB): track 0.00 -> 7.43 mm
- net +5V: track 0.00 -> 6.82 mm, vias 0 -> 3
- net Net-(U202-SW): track 0.00 -> 3.55 mm
- net Net-(J201-Pin_1): track 0.00 -> 3.38 mm
- added copper zone on In2.Cu, net +12V
- added copper zone on In2.Cu, net +3V3
- added copper zone on In2.Cu, net +5V
- added copper zone on In1.Cu, net GND
Other:
- board size 60 x 50 mm -> 75.2 x 68.5 mm

Commit message: dod some of the layout
Parts:
- J502: footprint Connector_Molex:Molex_Micro-Fit_3.0_43045-0600_2x03_P3.00mm_Horizontal -> Connector_Molex:Molex_Micro-Fit_3.0_43045-0621_2x03-1MP_P3.00mm_Horizontal
- SW301, SW302: footprint Button_Switch_SMD:SW_SPST_TL3342 -> Button_Switch_THT:SW_PUSH_6mm
- moved C501 121.5 mm to (73.6, 72.0), turned to 180 degrees
- moved C304 117.5 mm to (73.6, 69.0)
- moved C303 116.3 mm to (83.5, 64.0), turned to -90 degrees
- moved C305 114.8 mm to (78.0, 69.0)
- moved R303 103.5 mm to (83.5, 69.0), turned to 90 degrees
- moved C302 102.6 mm to (81.0, 47.5), turned to -90 degrees
- moved C301 101.7 mm to (81.0, 43.5), turned to 90 degrees
- moved C306 101.5 mm to (68.5, 59.0)
- moved R301 100.7 mm to (81.0, 60.6), turned to 90 degrees
- moved R302 97.9 mm to (93.5, 58.4), turned to 90 degrees
- moved C201 94.9 mm to (68.0, 65.5), turned to 90 degrees
- moved R305 93.2 mm to (74.5, 65.4), turned to 90 degrees
- moved JP501 90.3 mm to (111.5, 38.4), turned to -90 degrees
- moved R304 82.8 mm to (81.0, 51.4), turned to 90 degrees
- moved R_CAN_TERM501 78.5 mm to (111.5, 34.6), turned to -90 degrees
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Routing:
- net /COMMS/IO0: track 0.00 -> 86.0 mm
- net /COMMS/U0TXD: track 0.00 -> 83.2 mm, vias 0 -> 3
- net /COMMS/ESP32_EN: track 0.00 -> 81.9 mm, vias 0 -> 4
- net +12V: track 9.91 -> 81.1 mm
- net /COMMS/U0RXD: track 0.00 -> 58.1 mm
- net GND: track 16.0 -> 73.7 mm, vias 8 -> 15
- net +3V3: track 0.00 -> 37.5 mm, vias 0 -> 4
- net /COMMS/CAN_RX: track 0.00 -> 32.3 mm, vias 0 -> 2
- net /COMMS/CANH: track 0.00 -> 29.6 mm, vias 0 -> 2
- net /COMMS/INTERBOARD_TX: track 0.00 -> 28.2 mm
- net /COMMS/CANL: track 0.00 -> 28.1 mm
- net /COMMS/CAN_TX: track 0.00 -> 25.5 mm, vias 0 -> 2
- net Net-(U202-VBST): track 0.00 -> 23.8 mm
- net /COMMS/INTERBOARD_RX: track 0.00 -> 19.7 mm
- net +5V: track 6.82 -> 26.0 mm, vias 3 -> 1
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Other:
- board size 75.2 x 68.5 mm -> 64.5 x 51 mm

Commit message: fixed andrews layout
Parts:
- removed J301: Conn_01x06_Socket, Connector_PinHeader_2.54mm:PinHeader_1x06_P2.54mm_Vertical_SMD_Pin1Left
- added REF**: TestPoint_Pad_1.5x1.5mm, TestPoint:TestPoint_Pad_1.5x1.5mm, F.Cu at (51.7, 111.6)
- added REF**: TestPoint_Pad_1.5x1.5mm, TestPoint:TestPoint_Pad_1.5x1.5mm, F.Cu at (59.2, 111.6)
- added REF**: TestPoint_Pad_1.5x1.5mm, TestPoint:TestPoint_Pad_1.5x1.5mm, F.Cu at (56.7, 111.6)
- added REF**: TestPoint_Pad_1.5x1.5mm, TestPoint:TestPoint_Pad_1.5x1.5mm, F.Cu at (54.2, 111.6)
- added REF**: TestPoint_Pad_1.5x1.5mm, TestPoint:TestPoint_Pad_1.5x1.5mm, F.Cu at (61.7, 111.6)
- added REF**: TestPoint_Pad_1.5x1.5mm, TestPoint:TestPoint_Pad_1.5x1.5mm, F.Cu at (64.2, 111.6)
- moved U302 63.0 mm to (58.3, 115.8), turned to 180 degrees
- moved SW302 61.1 mm to (61.0, 105.2), turned to 90 degrees
- moved SW301 59.9 mm to (50.2, 105.0), turned to 90 degrees
- moved C203 56.8 mm to (44.5, 83.0)
- moved C301 56.8 mm to (44.5, 87.0)
- moved C302 56.8 mm to (44.5, 91.0)
- moved R304 56.8 mm to (44.5, 94.9)
- moved REF** 56.4 mm to (65.1, 116.8)
- moved C303 56.3 mm to (47.8, 107.5)
- moved J501 56.3 mm to (51.7, 108.5)
- moved REF** 56.3 mm to (80.2, 79.0)
- moved R_CAN_TERM501 56.3 mm to (75.8, 78.1)
- moved U501 56.3 mm to (71.3, 79.6)
- moved J503 56.3 mm to (76.6, 92.8)
- moved JP501 56.3 mm to (75.8, 81.8)
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Routing:
- net +12V: track 81.1 -> 11.2 mm, vias 4 -> 3
- net /COMMS/IO0: track 86.0 -> 29.3 mm
- net /COMMS/U0TXD: track 83.2 -> 37.0 mm, vias 3 -> 0
- net /COMMS/ESP32_EN: track 81.9 -> 48.9 mm, vias 4 -> 0
- net /COMMS/U0RXD: track 58.1 -> 36.6 mm
- net GND: track 73.7 -> 56.1 mm, vias 15 -> 13
- net Net-(U302-REGOUT): track 15.0 -> 0.00 mm
- net Net-(U302-SDA): track 10.7 -> 0.00 mm
- net Net-(U302-SCL): track 12.4 -> 1.75 mm, vias 2 -> 1
- net +3V3: track 37.5 -> 28.5 mm, vias 4 -> 3
- net Net-(U302-CPOUT): track 9.00 -> 0.00 mm
- net /COMMS/SYNC: track 18.6 -> 14.5 mm
- net /COMMS/CANL: track 28.1 -> 24.4 mm
- net /COMMS/CAN_RX: track 32.3 -> 30.4 mm
- net /COMMS/CAN_TX: track 25.5 -> 27.4 mm
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Other:
- board size 64.5 x 51 mm -> 59.2 x 46.8 mm
- board text added: "BOOT"
- board text added: "NIIIIGI IIGIGGGG JPM"
- board text added: "RESET"
