File: BajaBlaster/mcu.kicad_sch (KiCad schematic)
At the start: 16 parts, among them J301 Conn_01x06_Socket, SW301 SW_Push, SW302 SW_Push, U301 ESP32-WROOM-32, U302 MPU-6050

Commit message: small tweaks
Parts:
- J301: footprint Connector:Tag-Connect_TC2030-IDC-FP_2x03_P1.27mm_Vertical -> Connector_PinHeader_2.54mm:PinHeader_1x06_P2.54mm_Vertical_SMD_Pin1Left
Changed lines of the file:
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@@
 			)
 		)
-		(property "Footprint" "Connector:Tag-Connect_TC2030-IDC-FP_2x03_P1.27mm_Vertical"
+		(property "Footprint" "Connector_PinHeader_2.54mm:PinHeader_1x06_P2.54mm_Vertical_SMD_Pin1Left"
 			(at 60.325 168.275 0)
 			(hide yes)

Commit message: added power led indicator, double checked everything. passed erc
Parts:
- added D301: LED, LED_SMD:LED_0603_1608Metric, symbol Device:LED
- added R306: 1kOHM, symbol Device:R
- R303: value 10kOhm -> 10kOHM
Connections:
- net +3V3: now also R306.1
- net GND: now also D301.1 (K)
- new net: D301.2 (A), R306.2
Other:
- note added: "LOW VOLTAGE POWER LED"
