File: BajaBlaster/_restore_backup_2026-10-03T14-56-38-858/comms.kicad_sch (KiCad schematic)
At the start: 7 parts, among them J501 Conn_01x06_Pin, J502 INTERBOARD, J503 Conn_01x04_Pin, U501 TCAN330

Commit message: last touches before fabbing
Parts:
- J502: footprint Connector_Molex:Molex_Micro-Fit_3.0_43045-0610_2x03-1MP_P3.00mm_Horizontal -> Connector_Molex:Molex_Micro-Fit_3.0_43045-0600_2x03_P3.00mm_Horizontal
- J503: footprint Connector_Molex:Molex_Micro-Fit_3.0_43650-0412_1x04-1MP_P3.00mm_Horizontal -> Connector_Molex:Molex_Micro-Fit_3.0_43650-0410_1x04-1MP_P3.00mm_Horizontal
Changed lines of the file:
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@@
 			)
 		)
-		(property "Footprint" "Connector_Molex:Molex_Micro-Fit_3.0_43045-0610_2x03-1MP_P3.00mm_Horizontal"
+		(property "Footprint" "Connector_Molex:Molex_Micro-Fit_3.0_43045-0600_2x03_P3.00mm_Horizontal"
 			(at 99.695 37.465 0)
 			(hide yes)
@@
 			)
 		)
-		(property "Footprint" "Connector_Molex:Molex_Micro-Fit_3.0_43650-0412_1x04-1MP_P3.00mm_Horizontal"
+		(property "Footprint" "Connector_Molex:Molex_Micro-Fit_3.0_43650-0410_1x04-1MP_P3.00mm_Horizontal"
 			(at 156.845 37.465 0)
 			(hide yes)
